File: hardware/prism_mainboard/UnitB.kicad_sch (KiCad schematic)
At the start: 1 part, among them U1 XC7Z010-1CLG400C

Commit message: KiCAD Update
Added Power System Schematics. Decided on a 4 in 1 Buck and LDO, LP87222TQ1, for 3.3V and 1.8V LDO, and 1.8V and 1.0V Buck converter.
Parts:
- U1: footprint CLG400_XIL -> XC7Z010-1CLG400C:CLG400_XIL
Changed lines of the file:
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@@
 (kicad_sch
-	(version 20250114)
+	(version 20260306)
 	(generator "eeschema")
-	(generator_version "9.0")
+	(generator_version "10.0")
 	(paper "A4")
 	(global_label "VCCPINT"
@@
 		(property "Intersheetrefs" "${INTERSHEET_REFS}"
 			(at 99.6867 63.5 0)
+			(hide yes)
+			(show_name no)
+			(do_not_autoplace no)
 			(effects
 				(font
@@
 				)
 				(justify left)
-				(hide yes)
 			)
 		)
@@
 		(property "Intersheetrefs" "${INTERSHEET_REFS}"
 			(at 99.6867 88.9 0)
+			(hide yes)
+			(show_name no)
+			(do_not_autoplace no)
 			(effects
 				(font
@@
 				)
 				(justify left)
-				(hide yes)
 			)
 		)
@@
 		(property "Intersheetrefs" "${INTERSHEET_REFS}"
 			(at 99.6867 109.22 0)
+			(hide yes)
+			(show_name no)
+			(do_not_autoplace no)
 			(effects
 				(font
@@
 				)
 				(justify left)
-				(hide yes)
 			)
 		)
@@
 		(at 88.9 27.94 0)
 		(unit 2)
+		(body_style 1)
 		(exclude_from_sim no)
 		(in_bom yes)
 		(on_board yes)
+		(in_pos_files yes)
 		(dnp no)
 		(fields_autoplaced yes)
 		(property "Reference" "U1"
 			(at 137.16 17.78 0)
+			(show_name no)
+			(do_not_autoplace no)
 			(effects
 				(font
@@
 		(property "Value" "XC7Z010-1CLG400C"
 			(at 137.16 20.32 0)
+			(show_name no)
+			(do_not_autoplace no)
 			(effects
 				(font
@@
 			)
 		)
-		(property "Footprint" "CLG400_XIL"
+		(property "Footprint" "XC7Z010-1CLG400C:CLG400_XIL"
 			(at 88.9 27.94 0)
+			(hide yes)
+			(show_name no)
+			(do_not_autoplace no)
 			(effects
 				(font
@@
 					(italic yes)
 				)
-				(hide yes)
 			)
 		)
 		(property "Datasheet" "XC7Z010-1CLG400C"
 			(at 88.9 27.94 0)
+			(hide yes)
+			(show_name no)
+			(do_not_autoplace no)
 			(effects
 				(font
@@
 					(italic yes)
 				)
-				(hide yes)
 			)
 		)
 		(property "Description" ""
 			(at 88.9 27.94 0)
+			(hide yes)
+			(show_name no)
+			(do_not_autoplace no)
 			(effects
 				(font
 					(size 1.27 1.27)
 				)
-				(hide yes)
 			)
 		)
