File: hardware/prism_mainboard/UnitC.kicad_sch (KiCad schematic)
At the start: 3 parts, among them U1 XC7Z015-2CLG485I

Commit message: Updates
Mostly Schematic updates, nothing too big. Added a few datasheets
Connections:
- net USB_D3: now reaches U1.B11 (PS_MIO34_501)
- net SD_D1: now reaches U1.B12 (PS_MIO43_501)
- net SD_D3: now reaches U1.B14 (PS_MIO45_501)
- net USB_D7: now reaches U1.C10 (PS_MIO39_501)
- net SD_CMD: now reaches U1.C15 (PS_MIO41_501)
- net USB_D0: now reaches U1.C16 (PS_MIO32_501)
- net SD_SWITCH: now reaches U1.D11 (PS_MIO46_501)
- net SD_D0: now reaches U1.D15 (PS_MIO42_501)
- net SD_D2: now reaches U1.E10 (PS_MIO44_501)
- net DIR: now reaches U1.E15 (PS_MIO29_501)
- net USB_D6: now reaches U1.F10 (PS_MIO38_501)
- net NXT: now reaches U1.F14 (PS_MIO31_501)
- net USB_D2: now reaches U1.G11 (PS_MIO33_501)
