File: hardware/prism_mainboard/Power_System.kicad_sch (KiCad schematic)
At the start: 43 parts, among them IC1 LP875610RNFTQ1

Commit message: A whole lotta updates
Yeah
Parts:
- removed C8: 22uF, Capacitor_SMD:C_1206_3216Metric, symbol Device:C
- added C14, C43, C45, C47: 47uF, Capacitor_SMD:C_1206_3216Metric, symbol Device:C
- added C15, C44, C46: 22uF, Capacitor_SMD:C_1206_3216Metric, symbol Device:C
- added C42: 100nF, Capacitor_SMD:C_0201_0603Metric, symbol Device:C
- added L3, L4: 0.47uH, Inductor_SMD:L_Vishay_IHLP-1616, symbol Device:L
- added R3: 10k, symbol Device:R
- C11: value 4.7uF -> 10uF
- C12: value 2.2uF -> 10uF; footprint Capacitor_SMD:C_0201_0603Metric -> Capacitor_SMD:C_0805_2012Metric
- C41: value 2.2uF -> 100nF; footprint Capacitor_SMD:C_0201_0603Metric -> Capacitor_SMD:C_01005_0402Metric
- IC1: value LP875610RNFTQ1 -> LP87564WRNFTQ1
- L1, L2: footprint Inductor_SMD:L_0805_2012Metric -> Inductor_SMD:L_Vishay_IHLP-1616
Connections:
- net +1V8: now also IC1.1 (FB_B2_1), IC1.14 (FB_B1_1), IC1.21 (FB_B3_1), IC1.8 (FB_B0_1), L1.2, C14.1, C15.1, C43.1, C44.1, C45.1, C46.1, C47.1, L3.2, L4.2
- net GND: now also C14.2, C15.2, C42.2, C43.2, C44.2, C45.2, C46.2, C47.2, R3.2
- net SW_B1: now reaches L2.1
- net SW_B1: now also IC1.12 (SW_B1)
- net SW__B0: now reaches IC1.10 (SW_B0), L1.1
- net EN2: now reaches IC1.15 (EN2)
- net PGD_S: now reaches IC1.16 (PGOOD)
- net at IC1.19 (NINT): now also R3.1
- net EN3: now reaches IC1.2 (EN3)
- net PMIC_RST: now reaches IC1.20 (NRST)
- net SW_B3: now reaches IC1.23 (SW_B3)
- net SW_B3: now also L4.1
- net SW_B2: now reaches IC1.25 (SW_B2)
- net SW_B2: now also L3.1
- net CLK_IN_PS: now reaches IC1.3 (CLKIN)
- net SCL: now reaches IC1.5 (SCL)
- net SDA: now reaches IC1.6 (SDA)
- net EN1: now reaches IC1.7 (EN1)
- net VCC_Batt renamed VANA
- net VANA: now also C42.1
Other:
- moved on the sheet: C, C1, C10, C16, C17, C18, C19, C2, C20, C21, C22, C23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
