File: hardware/prism_mainboard/Power_System.kicad_sch (KiCad schematic)
At the start: 32 parts, among them U3 LP873222RHDRQ1, U4 100uF, U5 0.47uF, U6 4.7uF, U7 GND

Commit message: Origin Update
origin update
Parts:
- removed C27, C28: 22uF, ProtoFlow.pretty:C0805, symbol Device:C
- added U10: 0.47uF, symbol Device:C
- added U11: 100uF, symbol Device:C
- added U8: 4.7uF, symbol Device:C
- added U9: GND, symbol power:GND
Connections:
- net VCCAUX: now also U4.1, U5.1, U6.1, U10.1, U11.1, U8.1
- net at U3.18 (SDA), U3.9 (INT_N): no longer U3.17 (SCL)
- new net: U10.2, U11.2, U8.2, U9.1
Other:
- moved on the sheet: C24, C25, C26, U4, U5, U6
