File: hardware/prism_mainboard/prism_mainboard.kicad_sch (KiCad schematic)
At the start: 0 parts

Commit message: Zynq-7000 Schematic Updates
Added basic power net labels for the PL and PS portions of the FPGA.
Other:
- sheet Power_System renamed Power and Decoupling
- added sheet Data (data.kicad_sch)
- added sheet control (controls.kicad_sch)
Changed lines of the file:
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@@
+	)
+	(sheet
+		(at 19.05 101.6)
+		(size 85.09 3.81)
+		(exclude_from_sim no)
+		(in_bom yes)
+		(on_board yes)
+		(dnp no)
+		(fields_autoplaced yes)
+		(stroke
+			(width 0.1524)
+			(type solid)
+		)
+		(fill
+			(color 0 0 0 0)
+		)
+		(property "Sheetname" "Data"
+			(at 19.05 100.8884 0)
+			(show_name no)
+			(do_not_autoplace no)
+			(effects
+				(font
+					(size 1.27 1.27)
+				)
+				(justify left bottom)
+			)
+		)
+		(property "Sheetfile" "data.kicad_sch"
+			(at 19.05 105.9946 0)
+			(show_name no)
+			(do_not_autoplace no)
+			(effects
+				(font
+					(size 1.27 1.27)
+				)
+				(justify left top)
+			)
+		)
+		(instances
+			(project "prism_mainboard"
+				(path "/1d5f25f9-3e6f-41df-a8ec-41fc885bea9a"
+					(page "11")
+				)
+			)
+		)
 	)
 	(sheet
@@
 			(color 0 0 0 0)
 		)
-		(property "Sheetname" "Power_System"
+		(property "Sheetname" "Power and Decoupling"
 			(at 19.05 65.3284 0)
 			(show_name no)
@@
 				)
 			)
+		)
+	)
+	(sheet
+		(at 19.05 110.49)
+		(size 85.09 3.81)
+		(exclude_from_sim no)
+		(in_bom yes)
+		(on_board yes)
+		(dnp no)
+		(fields_autoplaced yes)
+		(stroke
+			(width 0.1524)
+			(type solid)
+		)
+		(fill
+			(color 0 0 0 0)
+		)
+		(property "Sheetname" "control"
+			(at 19.05 109.7784 0)
+			(show_name no)
+			(do_not_autoplace no)
+			(effects
+				(font
+					(size 1.27 1.27)
+				)
+				(justify left bottom)
+			)
+		)
+		(property "Sheetfile" "controls.kicad_sch"
+			(at 19.05 114.8846 0)
+			(show_name no)
+			(do_not_autoplace no)
+			(effects
+				(font
+					(size 1.27 1.27)
+				)
+				(justify left top)
+			)
+		)
+		(instances
+			(project "prism_mainboard"
+				(path "/1d5f25f9-3e6f-41df-a8ec-41fc885bea9a"
+					(page "12")
+				)
+			)

Commit message: Mainboard Updates
Started a lot of the basic schematic nets like GND and Power nets. Major Change: Decided on using the XC7Z015-1CLG485I instead of the 7010 or 7020 due to the ability to use HDMI interfaces with an adapter and more LUTs. Updated schematic symbols and footprints accordingly. Added Memory, Encoder, MicroSD schematics. Added LimeSDR footprints as well. Will Try to add Power to the entire board next.
Other:
- added sheet Data 2 (data2.kicad_sch)
- added sheet UnitE (xc7z015unit3.kicad_sch)
Changed lines of the file:
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@@
 			(project "prism_mainboard"
 				(path "/1d5f25f9-3e6f-41df-a8ec-41fc885bea9a"
-					(page "7")
+					(page "13")
 				)
 			)
@@
 	)
 	(sheet
+		(at 19.05 128.905)
+		(size 85.09 3.81)
+		(exclude_from_sim no)
+		(in_bom yes)
+		(on_board yes)
+		(dnp no)
+		(fields_autoplaced yes)
+		(stroke
+			(width 0.1524)
+			(type solid)
+		)
+		(fill
+			(color 0 0 0 0)
+		)
+		(property "Sheetname" "Data 2"
+			(at 19.05 128.1934 0)
+			(show_name no)
+			(do_not_autoplace no)
+			(effects
+				(font
+					(size 1.27 1.27)
+				)
+				(justify left bottom)
+			)
+		)
+		(property "Sheetfile" "data2.kicad_sch"
+			(at 19.05 133.2996 0)
+			(show_name no)
+			(do_not_autoplace no)
+			(effects
+				(font
+					(size 1.27 1.27)
+				)
+				(justify left top)
+			)
+		)
+		(instances
+			(project "prism_mainboard"
+				(path "/1d5f25f9-3e6f-41df-a8ec-41fc885bea9a"
+					(page "12")
+				)
+			)
+		)
+	)
+	(sheet
 		(at 19.05 93.98)
 		(size 85.09 3.81)
@@
 			(project "prism_mainboard"
 				(path "/1d5f25f9-3e6f-41df-a8ec-41fc885bea9a"
-					(page "12")
-				)
-			)
+					(page "14")
+				)
+			)
+		)
+	)
+	(sheet
+		(at 19.05 120.65)
+		(size 85.09 3.81)
+		(exclude_from_sim no)
+		(in_bom yes)
+		(on_board yes)
+		(dnp no)
+		(fields_autoplaced yes)
+		(stroke
+			(width 0.1524)
+			(type solid)
+		)
+		(fill
+			(color 0 0 0 0)
+		)
+		(property "Sheetname" "UnitE"
+			(at 19.05 119.9384 0)
+			(show_name no)
+			(do_not_autoplace no)
+			(effects
+				(font
+					(size 1.27 1.27)
+				)
+				(justify left bottom)
+			)
+		)
+		(property "Sheetfile" "xc7z015unit3.kicad_sch"
+			(at 19.05 125.0446 0)
+			(show_name no)
+			(do_not_autoplace no)
+			(effects
+				(font
+					(size 1.27 1.27)
+				)
+				(justify left top)
+			)
+		)
+		(instances
+			(project "prism_mainboard"
+				(path "/1d5f25f9-3e6f-41df-a8ec-41fc885bea9a"
+					(page "7")
+				)
+			)
