File: hardware/prism_mainboard/xc7z015unit3.kicad_sch (KiCad schematic)
At the start: 1 part, among them U1 XC7Z015-2CLG485I

Commit message: Schematic Updates
Updated the DDR3 DRAM to 4Gb, added a lot of nets and started updating the power and decoupling components. Updated .gitignore to avoid .mkv files.
Connections:
- net VCCO_DDR: now reaches U1.R21 (VCCO_DDR_502)
- net VCCO_DDR: now also U1.V22 (VCCO_DDR_502)
Changed lines of the file:
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@@
+		)
+	)
+	(global_label "VCCO_DDR"
+		(shape input)
+		(at 74.93 40.64 180)
+		(fields_autoplaced yes)
+		(effects
+			(font
+				(size 1.27 1.27)
+			)
+			(justify right)
+		)
+		(property "Intersheetrefs" "${INTERSHEET_REFS}"
+			(at 62.2081 40.64 0)
+			(hide yes)
+			(show_name no)
+			(do_not_autoplace no)
+			(effects
+				(font
+					(size 1.27 1.27)
+				)
+				(justify right)
+			)
 		)
 	)
@@
 			(hide yes)
 			(show_name no)
+			(do_not_autoplace no)
+			(effects
+				(font
+					(size 1.27 1.27)
+				)
+				(justify right)
+			)
+		)
+	)
+	(global_label "VCCO_DDR"
+		(shape input)
+		(at 74.93 142.24 180)
+		(fields_autoplaced yes)
+		(effects
+			(font
+				(size 1.27 1.27)
+			)
+			(justify right)
+		)
+		(property "Intersheetrefs" "${INTERSHEET_REFS}"
+			(at 62.2081 142.24 0)
+			(hide yes)
+			(show_name no)
