File: hardware/prism_mainboard/_autosave-prism_mainboard.kicad_pcb (KiCad board)
At the start: 6 copper layers, 100 x 100 mm, 76 parts, among them IC1 KTDM4G3C618BGIEAT, IC2 KTDM4G3C618BGIEAT, IC3 USB3320C-EZK, J1 503398-1892, U1 XC7Z015-2CLG485I, U2 LMS7002M, U3 PEC16-4220F-S0024, U4 AMS1117-1.8, U5 AMS1117-1.8, U6 AMS1117-1.8, U7 AMS1117-1.8

Commit message: Schematic Updates & PCB Population
Populated the PCB with footprints from Main PC, should show up now. Also been updating the KiCAD schematics to connect the DDR3L Modules to the FPGA. Should be done except for a few pins that I'm not sure what they do yet. But Addressing and data pins should be connected correctly now
Connections:
- IC1 pad A2: unconnected-(IC1-DQU5-PadA2) -> DQU5_0
- IC1 pad A3: unconnected-(IC1-DQU7-PadA3) -> DQU7_0
- IC1 pad A7: unconnected-(IC1-DQU4-PadA7) -> DQU4_0
- IC1 pad B7: unconnected-(IC1-~{DQSU}-PadB7) -> DQSUN_0
- IC1 pad B8: unconnected-(IC1-DQU6-PadB8) -> DQU6_0
- IC1 pad C2: unconnected-(IC1-DQU3-PadC2) -> DQU3_0
- IC1 pad C3: unconnected-(IC1-DQU1-PadC3) -> DQU1_0
- IC1 pad C7: unconnected-(IC1-DQSU-PadC7) -> DQSUP_0
- IC1 pad C8: unconnected-(IC1-DQU2-PadC8) -> DQU2_0
- IC1 pad D3: unconnected-(IC1-DMU-PadD3) -> DM1
- IC1 pad D7: unconnected-(IC1-DQU0-PadD7) -> DQU0_0
- IC1 pad E3: unconnected-(IC1-DQL0-PadE3) -> DQL0_0
- IC1 pad E7: unconnected-(IC1-DML-PadE7) -> DM0
- IC1 pad F2: unconnected-(IC1-DQL2-PadF2) -> DQL2_0
- IC1 pad F3: unconnected-(IC1-DQSL-PadF3) -> DQSLP_0
- IC1 pad F7: unconnected-(IC1-DQL1-PadF7) -> DQL1_0
- IC1 pad F8: unconnected-(IC1-DQL3-PadF8) -> DQL3_0
- IC1 pad G2: unconnected-(IC1-DQL6-PadG2) -> DQL6_0
- IC1 pad G3: unconnected-(IC1-~{DQSL}-PadG3) -> DQSLN_0
- IC1 pad H3: unconnected-(IC1-DQL4-PadH3) -> DQL4_0
- IC1 pad H7: unconnected-(IC1-DQL7-PadH7) -> DQL7_0
- IC1 pad H8: unconnected-(IC1-DQL5-PadH8) -> DQL5_0
- IC1 pad J3: unconnected-(IC1-~{RAS}-PadJ3) -> RAS
- IC1 pad J7: unconnected-(IC1-CK-PadJ7) -> CKP
- IC1 pad K1: unconnected-(IC1-ODT-PadK1) -> ODT
- IC1 pad K3: unconnected-(IC1-~{CAS}-PadK3) -> CAS
- IC1 pad K7: unconnected-(IC1-~{CK}-PadK7) -> CKN
- IC1 pad K9: unconnected-(IC1-CKE-PadK9) -> CKE
- IC1 pad L2: unconnected-(IC1-~{CS}-PadL2) -> CS
- IC1 pad L3: unconnected-(IC1-~{WE}-PadL3) -> WE
- IC1 pad L7: unconnected-(IC1-A10/AP-PadL7) -> A10
- IC1 pad M2: unconnected-(IC1-BA0-PadM2) -> BA0
- IC1 pad M3: unconnected-(IC1-BA2-PadM3) -> BA
- IC1 pad N2: unconnected-(IC1-A3-PadN2) -> A3
- IC1 pad N3: unconnected-(IC1-A0-PadN3) -> A0
- IC1 pad N7: unconnected-(IC1-A12/~{BC}-PadN7) -> A12
- IC1 pad N8: unconnected-(IC1-BA1-PadN8) -> BA1
- IC1 pad P2: unconnected-(IC1-A5-PadP2) -> A5
- IC1 pad P3: unconnected-(IC1-A2-PadP3) -> A2
- IC1 pad P7: unconnected-(IC1-A1-PadP7) -> A1
- IC1 pad P8: unconnected-(IC1-A4-PadP8) -> A4
- IC1 pad R2: unconnected-(IC1-A7-PadR2) -> A7
- IC1 pad R3: unconnected-(IC1-A9-PadR3) -> A9
- IC1 pad R7: unconnected-(IC1-A11-PadR7) -> A11
- IC1 pad R8: unconnected-(IC1-A6-PadR8) -> A6
- IC1 pad T3: unconnected-(IC1-A13-PadT3) -> A13
- IC1 pad T7: unconnected-(IC1-A14-PadT7) -> A14
- IC1 pad T8: unconnected-(IC1-A8-PadT8) -> A8
- IC2 pad A2: unconnected-(IC2-DQU5-PadA2) -> DQU5_1
- IC2 pad A3: unconnected-(IC2-DQU7-PadA3) -> DQU7_1
- IC2 pad A7: unconnected-(IC2-DQU4-PadA7) -> DQU4_1
- IC2 pad B7: unconnected-(IC2-~{DQSU}-PadB7) -> DQSUN_1
- IC2 pad B8: unconnected-(IC2-DQU6-PadB8) -> DQU6_1
- IC2 pad C2: unconnected-(IC2-DQU3-PadC2) -> DQU3_1
- IC2 pad C3: unconnected-(IC2-DQU1-PadC3) -> DQU1_1
- IC2 pad C7: unconnected-(IC2-DQSU-PadC7) -> DQSUP_1
- IC2 pad C8: unconnected-(IC2-DQU2-PadC8) -> DQU2_1
- IC2 pad D3: unconnected-(IC2-DMU-PadD3) -> DM3
- IC2 pad D7: unconnected-(IC2-DQU0-PadD7) -> DQU0_1
- IC2 pad E3: unconnected-(IC2-DQL0-PadE3) -> DQL0_1
- IC2 pad E7: unconnected-(IC2-DML-PadE7) -> DM2
- IC2 pad F2: unconnected-(IC2-DQL2-PadF2) -> DQL2_1
- IC2 pad F3: unconnected-(IC2-DQSL-PadF3) -> DQSLP_1
- IC2 pad F7: unconnected-(IC2-DQL1-PadF7) -> DQL1_1
- IC2 pad F8: unconnected-(IC2-DQL3-PadF8) -> DQL3_1
- IC2 pad G2: unconnected-(IC2-DQL6-PadG2) -> DQL6_1
- IC2 pad G3: unconnected-(IC2-~{DQSL}-PadG3) -> DQSLN_1
- IC2 pad H3: unconnected-(IC2-DQL4-PadH3) -> DQL4_1
- IC2 pad H7: unconnected-(IC2-DQL7-PadH7) -> DQL7_1
- IC2 pad H8: unconnected-(IC2-DQL5-PadH8) -> DQL5_1
- IC2 pad J3: unconnected-(IC2-~{RAS}-PadJ3) -> RAS
- IC2 pad J7: unconnected-(IC2-CK-PadJ7) -> CKP
- IC2 pad K1: unconnected-(IC2-ODT-PadK1) -> ODT
- IC2 pad K3: unconnected-(IC2-~{CAS}-PadK3) -> CAS
- IC2 pad K7: unconnected-(IC2-~{CK}-PadK7) -> CKN
- IC2 pad K9: unconnected-(IC2-CKE-PadK9) -> CKE
- IC2 pad L2: unconnected-(IC2-~{CS}-PadL2) -> CS
- IC2 pad L3: unconnected-(IC2-~{WE}-PadL3) -> WE
- IC2 pad L7: unconnected-(IC2-A10/AP-PadL7) -> A10
- IC2 pad M2: unconnected-(IC2-BA0-PadM2) -> BA0
- IC2 pad M3: unconnected-(IC2-BA2-PadM3) -> BA
- IC2 pad N2: unconnected-(IC2-A3-PadN2) -> A3
- IC2 pad N3: unconnected-(IC2-A0-PadN3) -> A0
- IC2 pad N7: unconnected-(IC2-A12/~{BC}-PadN7) -> A12
- IC2 pad N8: unconnected-(IC2-BA1-PadN8) -> BA1
- IC2 pad P2: unconnected-(IC2-A5-PadP2) -> A5
- IC2 pad P3: unconnected-(IC2-A2-PadP3) -> A2
- IC2 pad P7: unconnected-(IC2-A1-PadP7) -> A1
- IC2 pad P8: unconnected-(IC2-A4-PadP8) -> A4
- IC2 pad R2: unconnected-(IC2-A7-PadR2) -> A7
- IC2 pad R3: unconnected-(IC2-A9-PadR3) -> A9
- IC2 pad R7: unconnected-(IC2-A11-PadR7) -> A11
- IC2 pad R8: unconnected-(IC2-A6-PadR8) -> A6
- IC2 pad T3: unconnected-(IC2-A13-PadT3) -> A13
- IC2 pad T7: unconnected-(IC2-A14-PadT7) -> A14
- IC2 pad T8: unconnected-(IC2-A8-PadT8) -> A8
- U1 pad AA22: unconnected-(U1E-PS_DDR_DQ26_502-PadAA22) -> DQU2_1
- U1 pad B21: unconnected-(U1C-PS_DDR_DQ2_502-PadB21) -> DQL2_0
- U1 pad B22: unconnected-(U1C-PS_DDR_DM0_502-PadB22) -> DM0
- U1 pad C20: unconnected-(U1C-PS_DDR_DQ1_502-PadC20) -> DQL1_0
- U1 pad C21: unconnected-(U1C-PS_DDR_DQS_P0_502-PadC21) -> DQSLP_0
- U1 pad D20: unconnected-(U1C-PS_DDR_DQ3_502-PadD20) -> DQL3_0
- U1 pad D21: unconnected-(U1C-PS_DDR_DQS_N0_502-PadD21) -> DQSLN_0
- U1 pad D22: unconnected-(U1C-PS_DDR_DQ0_502-PadD22) -> DQL0_0
- U1 pad E20: unconnected-(U1C-PS_DDR_DQ4_502-PadE20) -> DQL4_0
- U1 pad E22: unconnected-(U1C-PS_DDR_DQ5_502-PadE22) -> DQL5_0
- U1 pad F16: unconnected-(U1C-PS_CLK_500-PadF16) -> CLK
- U1 pad F19: unconnected-(U1C-PS_DDR_A13_502-PadF19) -> A13
- U1 pad F21: unconnected-(U1C-PS_DDR_DQ6_502-PadF21) -> DQL6_0
- U1 pad F22: unconnected-(U1C-PS_DDR_DQ7_502-PadF22) -> DQL7_0
- U1 pad G18: unconnected-(U1C-PS_DDR_A11_502-PadG18) -> A11
- U1 pad G19: unconnected-(U1C-PS_DDR_A14_502-PadG19) -> A14
- U1 pad G21: unconnected-(U1C-PS_DDR_DQ8_502-PadG21) -> DQU0_0
- U1 pad G22: unconnected-(U1C-PS_DDR_DQ9_502-PadG22) -> DQU1_0
- U1 pad H18: unconnected-(U1D-PS_DDR_A9_502-PadH18) -> A9
- U1 pad H19: unconnected-(U1D-PS_DDR_A12_502-PadH19) -> A12
- U1 pad H21: unconnected-(U1D-PS_DDR_DQS_P1_502-PadH21) -> DQSUP_0
- U1 pad J16: unconnected-(U1D-PS_DDR_A6_502-PadJ16) -> A6
- U1 pad J17: unconnected-(U1D-PS_DDR_A7_502-PadJ17) -> A7
- U1 pad J18: unconnected-(U1D-PS_DDR_A8_502-PadJ18) -> A8
- U1 pad J20: unconnected-(U1D-PS_DDR_A10_502-PadJ20) -> A10
- U1 pad J21: unconnected-(U1D-PS_DDR_DQS_N1_502-PadJ21) -> DQSUN_0
- U1 pad J22: unconnected-(U1D-PS_DDR_DQ14_502-PadJ22) -> DQU6_0
- U1 pad K17: unconnected-(U1D-PS_DDR_A4_502-PadK17) -> A4
- U1 pad K18: unconnected-(U1D-PS_DDR_A5_502-PadK18) -> A5
- U1 pad K19: unconnected-(U1D-PS_DDR_A2_502-PadK19) -> A2
- U1 pad K20: unconnected-(U1D-PS_DDR_DQ15_502-PadK20) -> DQU7_0
- U1 pad K22: unconnected-(U1D-PS_DDR_DQ13_502-PadK22) -> DQU5_0
- U1 pad L16: unconnected-(U1D-PS_DDR_BA0_502-PadL16) -> BA0
- U1 pad L17: unconnected-(U1D-PS_DDR_BA1_502-PadL17) -> BA1
- U1 pad L19: unconnected-(U1D-PS_DDR_A3_502-PadL19) -> A3
- U1 pad L20: unconnected-(U1D-PS_DDR_DQ12_502-PadL20) -> DQU4_0
- U1 pad L21: unconnected-(U1D-PS_DDR_DQ11_502-PadL21) -> DQU3_0
- U1 pad L22: unconnected-(U1D-PS_DDR_DQ10_502-PadL22) -> DQU2_0
- U1 pad M17: unconnected-(U1D-PS_DDR_BA2_502-PadM17) -> BA2
- U1 pad M18: unconnected-(U1D-PS_DDR_A1_502-PadM18) -> A1
- U1 pad M19: unconnected-(U1D-PS_DDR_A0_502-PadM19) -> A0
- U1 pad M21: unconnected-(U1D-PS_DDR_DQ22_502-PadM21) -> DQL6_1
- U1 pad M22: unconnected-(U1D-PS_DDR_DQ16_502-PadM22) -> DQL0_1
- U1 pad N18: unconnected-(U1D-PS_DDR_CKN_502-PadN18) -> CKN
- U1 pad N19: unconnected-(U1D-PS_DDR_CKP_502-PadN19) -> CKP
- U1 pad N20: unconnected-(U1D-PS_DDR_DQ18_502-PadN20) -> DQL2_1
- U1 pad N21: unconnected-(U1D-PS_DDR_DQS_P2_502-PadN21) -> DQSLP_1
- U1 pad P17: unconnected-(U1D-PS_DDR_CS_B_502-PadP17) -> CS
- U1 pad P18: unconnected-(U1D-PS_DDR_ODT_502-PadP18) -> ODT
- U1 pad P20: unconnected-(U1D-PS_DDR_CAS_B_502-PadP20) -> CAS
- U1 pad P21: unconnected-(U1D-PS_DDR_DQS_N2_502-PadP21) -> DQSLN_1
- U1 pad P22: unconnected-(U1D-PS_DDR_DM2_502-PadP22) -> DM2
- U1 pad R18: unconnected-(U1E-PS_DDR_RAS_B_502-PadR18) -> RAS
- U1 pad R19: unconnected-(U1E-PS_DDR_WE_B_502-PadR19) -> WE
- U1 pad R20: unconnected-(U1E-PS_DDR_DQ20_502-PadR20) -> DQL4_1
- U1 pad R22: unconnected-(U1E-PS_DDR_DQ23_502-PadR22) -> DQL7_1
- U1 pad T19: unconnected-(U1E-PS_DDR_CKE_502-PadT19) -> CKE
- U1 pad T20: unconnected-(U1E-PS_DDR_DQ17_502-PadT20) -> DQL1_1
- U1 pad T21: unconnected-(U1E-PS_DDR_DQ21_502-PadT21) -> DQL5_1
- U1 pad T22: unconnected-(U1E-PS_DDR_DQ19_502-PadT22) -> DQL3_1
- U1 pad U21: unconnected-(U1E-PS_DDR_DQ27_502-PadU21) -> DQU3_1
- U1 pad U22: unconnected-(U1E-PS_DDR_DQ25_502-PadU22) -> DQU1_1
- U1 pad V20: unconnected-(U1E-PS_DDR_DQ30_502-PadV20) -> DQU6_1
- U1 pad V21: unconnected-(U1E-PS_DDR_DQS_P3_502-PadV21) -> DQSUP_1
- U1 pad W20: unconnected-(U1E-PS_DDR_DQ29_502-PadW20) -> DQU5_1
- U1 pad W21: unconnected-(U1E-PS_DDR_DQS_N3_502-PadW21) -> DQSUN_1
- U1 pad W22: unconnected-(U1E-PS_DDR_DQ28_502-PadW22) -> DQU4_1
- U1 pad Y20: unconnected-(U1E-PS_DDR_DQ24_502-PadY20) -> DQU0_1
- U1 pad Y22: unconnected-(U1E-PS_DDR_DQ31_502-PadY22) -> DQU7_1
