File: hardware/prism_mainboard/UnitA.kicad_sch (KiCad schematic)
At the start: 1 part, among them U1 XC7Z015-2CLG485I

Commit message: Updates
Mostly Schematic updates, nothing too big. Added a few datasheets
Connections:
- net USB_D5: now reaches U1.B9 (PS_MIO37_501)
- net SD_CLK: now reaches U1.E9 (PS_MIO40_501)
- net USB_D3: now reaches U1.F9 (PS_MIO35_501)
- net DIQ1_10 renamed DIQ1_D10
Changed lines of the file:
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@@
+		)
+	)
+	(global_label "USB_D3"
+		(shape input)
+		(at 203.2 138.43 0)
+		(fields_autoplaced yes)
+		(effects
+			(font
+				(size 1.27 1.27)
+			)
+			(justify left)
+		)
+		(property "Intersheetrefs" "${INTERSHEET_REFS}"
+			(at 213.4423 138.43 0)
+			(hide yes)
+			(show_name no)
+			(do_not_autoplace no)
+			(effects
+				(font
+					(size 1.27 1.27)
+				)
+				(justify left)
+			)
 		)
 	)
@@
 		)
 	)
+	(global_label "SD_CLK"
+		(shape input)
+		(at 81.28 140.97 180)
+		(fields_autoplaced yes)
+		(effects
+			(font
+				(size 1.27 1.27)
+			)
+			(justify right)
+		)
+		(property "Intersheetrefs" "${INTERSHEET_REFS}"
+			(at 71.2796 140.97 0)
+			(hide yes)
+			(show_name no)
+			(do_not_autoplace no)
+			(effects
+				(font
+					(size 1.27 1.27)
+				)
+				(justify right)
+			)
+		)
+	)
 	(global_label "DIQ2_D5"
 		(shape input)
@@
 		)
 	)
-	(global_label "DIQ1_10"
+	(global_label "DIQ1_D10"
 		(shape input)
 		(at 81.28 130.81 180)
@@
 		)
 		(property "Intersheetrefs" "${INTERSHEET_REFS}"
-			(at 70.4934 130.81 0)
+			(at 69.2234 130.81 0)
 			(hide yes)
 			(show_name no)
@@
 			)
 		)
+	)
+	(global_label "USB_D5"
+		(shape input)
+		(at 81.28 72.39 180)
+		(fields_autoplaced yes)
+		(effects
+			(font
+				(size 1.27 1.27)
+			)
+			(justify right)
+		)
+		(property "Intersheetrefs" "${INTERSHEET_REFS}"
+			(at 71.0377 72.39 0)
+			(hide yes)
+			(show_name no)
+			(do_not_autoplace no)
+			(effects
+				(font
+					(size 1.27 1.27)
+				)
+				(justify right)
+			)
+		)
