File: hardware/prism_mainboard/controls.kicad_sch (KiCad schematic)
At the start: 0 parts

Commit message: Mainboard Updates
Started a lot of the basic schematic nets like GND and Power nets. Major Change: Decided on using the XC7Z015-1CLG485I instead of the 7010 or 7020 due to the ability to use HDMI interfaces with an adapter and more LUTs. Updated schematic symbols and footprints accordingly. Added Memory, Encoder, MicroSD schematics. Added LimeSDR footprints as well. Will Try to add Power to the entire board next.
Parts:
- added U3: PEC16-4220F-S0024, PEC164120FS0012, symbol SamacSys:PEC16-4220F-S0024
Changed lines of the file:
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@@
 	(generator_version "10.0")
 	(paper "A4")
+	(symbol
+		(lib_id "SamacSys:PEC16-4220F-S0024")
+		(at 72.39 48.26 0)
+		(unit 1)
+		(body_style 1)
+		(exclude_from_sim no)
+		(in_bom yes)
+		(on_board yes)
+		(in_pos_files yes)
+		(dnp no)
+		(fields_autoplaced yes)
+		(property "Reference" "U3"
+			(at 105.41 41.8398 0)
+			(show_name no)
+			(do_not_autoplace no)
+			(effects
+				(font
+					(size 1.27 1.27)
+				)
+			)
+		)
+		(property "Value" "PEC16-4220F-S0024"
+			(at 105.41 44.3798 0)
+			(show_name no)
+			(do_not_autoplace no)
+			(effects
+				(font
+					(size 1.27 1.27)
+				)
+			)
+		)
+		(property "Footprint" "PEC164120FS0012"
+			(at 93.98 138.1 0)
+			(hide yes)
+			(show_name no)
+			(do_not_autoplace no)
+			(effects
+				(font
+					(size 1.27 1.27)
+				)
+				(justify left top)
+			)
+		)
+		(property "Datasheet" "https://www.bourns.com/pdfs/PEC16.pdf"
+			(at 93.98 238.1 0)
+			(hide yes)
+			(show_name no)
+			(do_not_autoplace no)
+			(effects
+				(font
+					(size 1.27 1.27)
+				)
+				(justify left top)
+			)
+		)
+		(property "Description" "Bourns Encoder 24ppr ppr 5 V dc"
+			(at 72.39 48.26 0)
+			(hide yes)
+			(show_name no)
+			(do_not_autoplace no)
+			(effects
+				(font
+					(size 1.27 1.27)
+				)
+			)
+		)
+		(property "Height" "28"
+			(at 93.98 438.1 0)
+			(hide yes)
+			(show_name no)
+			(do_not_autoplace no)
+			(effects
+				(font
+					(size 1.27 1.27)
+				)
+				(justify left top)
+			)
+		)
+		(property "Mouser Part Number" "652-PEC16-4220FS0024"
+			(at 93.98 538.1 0)
+			(hide yes)
+			(show_name no)
+			(do_not_autoplace no)
+			(effects
+				(font
+					(size 1.27 1.27)
+				)
+				(justify left top)
+			)
+		)
+		(property "Mouser Price/Stock" "https://www.mouser.co.uk/ProductDetail/Bourns/PEC16-4220F-S0024?qs=6FD5PBp7ZtQte%252Bg7b%2FiMUw%3D%3D"
+			(at 93.98 638.1 0)
+			(hide yes)
+			(show_name no)
+			(do_not_autoplace no)
+			(effects
+				(font
+					(size 1.27 1.27)
+				)
+				(justify left top)
+			)
+		)
+		(property "Manufacturer_Name" "Bourns"
+			(at 93.98 738.1 0)
+			(hide yes)
+			(show_name no)
+			(do_not_autoplace no)
+			(effects
+				(font
+					(size 1.27 1.27)
+				)
+				(justify left top)
+			)
+		)
+		(property "Manufacturer_Part_Number" "PEC16-4220F-S0024"
+			(at 93.98 838.1 0)
+			(hide yes)
+			(show_name no)
+			(do_not_autoplace no)
+			(effects
+				(font
+					(size 1.27 1.27)
+				)
+				(justify left top)
+			)
+		)
+		(pin "D1"
+		)
+		(pin "E1"
+		)
+		(pin "MH1"
+		)
+		(pin "C1"
+		)
+		(pin "B1"
+		)
+		(pin "MH2"
+		)
+		(pin "A1"
+		)
+		(instances
+			(project "prism_mainboard"
+				(path "/1d5f25f9-3e6f-41df-a8ec-41fc885bea9a/b7ee0d75-d597-42aa-b567-b6bd9aedde27"
+					(reference "U3")
+					(unit 1)
+				)
+			)
+		)
+	)
 )

Commit message: Updates
Mostly Schematic updates, nothing too big. Added a few datasheets
Parts:
- added J2: UJ32-21-C-H-G-HMT-LT-P24-TR, UJ3221CHGHMTLTP24TR, symbol SamacSys:UJ32-21-C-H-G-HMT-LT-P24-TR
- added R7, R8: 5.1k, symbol Device:R
- added U8: PEC16-4220F-S0024, PEC164120FS0012, symbol SamacSys:PEC16-4220F-S0024
Connections:
- new net: J2.A5 (CC1), R7.2
- new net: J2.B5 (CC2), R8.1
- new net DATA+: J2.A6 (DP1), J2.B6 (DP2)
- new net DATA-: J2.A7 (DN1), J2.B7 (DN2)
- new net GND: J2.A1 (GND_1), J2.A12 (GND_2), J2.B1 (GND_3), J2.B12 (GND_4), R7.1, R8.2
- new net VBUS: J2.A4 (VBUS_1), J2.A9 (VBUS_2), J2.B4 (VBUS_3), J2.B9 (VBUS_4)
Other:
- moved on the sheet: U3
