File: hardware/mainboard_PF/PRISM/XC7Z010-U2.kicad_sch (KiCad schematic)
At the start: 0 parts

Commit message: More Protoflow
Power Systesm
Parts:
- added U1: XC7Z010-1CLG400C, ProtoFlow.pretty:CLG400_XIL, symbol XC7Z010-1CLG400C
Changed lines of the file:
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@@
     (company "Protoflow")
+  )
+  (symbol (lib_id "XC7Z010-1CLG400C") (at 105.41 36.83 0)
+    (unit 2)
+    (convert 1)
+    (in_bom yes)
+    (on_board yes)
+    (property "Reference" "U1" (id 0) (at 114.3 30.48 0) (effects (font (size 1.524 1.524))))
+    (property "Value" "XC7Z010-1CLG400C" (id 1) (at 153.67 167.64 0) (effects (font (size 1.524 1.524))))
+    (property "Footprint" "ProtoFlow.pretty:CLG400_XIL" (id 2) (at 105.41 36.83 0) (effects (font (size 1.27 1.27)) hide))
+    (property "Datasheet" "XC7Z010-1CLG400C" (id 3) (at 105.41 36.83 0) (effects (font (size 1.27 1.27)) hide))
+    (property "Protoflow_Source" "kicad" (id 4) (at 105.41 36.83 0) (effects (font (size 1.27 1.27)) hide))
+    (pin "A10")
+    (pin "A11")
+    (pin "A12")
+    (pin "A13")
+    (pin "A14")
+    (pin "A15")
+    (pin "A16")
+    (pin "A17")
+    (pin "A18")
+    (pin "A19")
+    (pin "A20")
+    (pin "B10")
+    (pin "B11")
+    (pin "B12")
+    (pin "B13")
+    (pin "B14")
+    (pin "B15")
+    (pin "B16")
+    (pin "B17")
+    (pin "B18")
+    (pin "M2")
+    (pin "M3")
+    (pin "M4")
+    (pin "M5")
+    (pin "M6")
+    (pin "M7")
+    (pin "M8")
+    (pin "M9")
+    (pin "N1")
+    (pin "N2")
+    (pin "N3")
+    (pin "N4")
+    (pin "N5")
+    (pin "N6")
+    (pin "N7")
+    (pin "N8")
+    (pin "N9")
+    (pin "P1")
+    (pin "P2")
+    (pin "P3")
+    (pin "P4")
+    (pin "P5")
+    (pin "P6")
+    (pin "P7")
+    (pin "P8")
+    (pin "P9")
+    (pin "R1")
+    (pin "R2")
+    (pin "R3")
+    (pin "R4")
+    (pin "R5")
+    (pin "R6")
+    (pin "R7")
+    (pin "R8")
+    (pin "R9")
+    (pin "T1")
+    (pin "T2")
+    (pin "T3")
+    (pin "T4")
+    (pin "T5")
+    (pin "T6")
+    (pin "T7")
+    (pin "T8")
+    (pin "T9")
+    (pin "U1")
+    (pin "U2")
+    (pin "U3")
+    (pin "U4")
+    (pin "U5")
+    (pin "U6")
+    (pin "U7")
+    (pin "U8")
+    (pin "U9")
+    (pin "V1")
+    (pin "V2")
+    (pin "V3")
+    (pin "V4")
+    (pin "V5")
+    (pin "V6")
+    (pin "V7")
+    (pin "V8")
+    (pin "V9")
+    (pin "W1")
+    (pin "W2")
+    (pin "W3")
+    (pin "W4")
+    (pin "W5")
+    (pin "W6")
+    (pin "W7")
+    (pin "W8")
+    (pin "W9")
+    (pin "Y1")
+    (pin "Y2")
+    (pin "Y3")
+    (pin "Y4")
+    (pin "Y5")
+    (pin "Y6")
+    (pin "Y7")
+    (pin "Y8")
+    (pin "Y9")
+    (instances
+      (project "protoflow"
+        (path "/" (reference "U1") (unit 2))
+      )
+    )
   )
   (sheet_instances
