File: hardware/mainboard_PF/PRISM/XC7Z010-U3.kicad_sch (KiCad schematic)
At the start: 0 parts

Commit message: More Protoflow
Power Systesm
Parts:
- added U1: XC7Z010-1CLG400C, ProtoFlow.pretty:CLG400_XIL, symbol XC7Z010-1CLG400C
Other:
- title: Untitled -> XC7Z010-U3
Changed lines of the file:
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@@
   (paper "A4")
   (title_block
-    (title "Untitled")
+    (title "XC7Z010-U3")
     (rev "1.0")
     (company "Protoflow")
   )
+  (symbol (lib_id "XC7Z010-1CLG400C") (at 92.71 38.1 0)
+    (unit 3)
+    (convert 1)
+    (in_bom yes)
+    (on_board yes)
+    (property "Reference" "U1" (id 0) (at 101.6 31.75 0) (effects (font (size 1.524 1.524))))
+    (property "Value" "XC7Z010-1CLG400C" (id 1) (at 153.67 168.91 0) (effects (font (size 1.524 1.524))))
+    (property "Footprint" "ProtoFlow.pretty:CLG400_XIL" (id 2) (at 92.71 38.1 0) (effects (font (size 1.27 1.27)) hide))
+    (property "Datasheet" "XC7Z010-1CLG400C" (id 3) (at 92.71 38.1 0) (effects (font (size 1.27 1.27)) hide))
+    (property "Protoflow_Source" "kicad" (id 4) (at 92.71 38.1 0) (effects (font (size 1.27 1.27)) hide))
+    (pin "B19")
+    (pin "B20")
+    (pin "C10")
+    (pin "C11")
+    (pin "C12")
+    (pin "C13")
+    (pin "C14")
+    (pin "C15")
+    (pin "C16")
+    (pin "C17")
+    (pin "C18")
+    (pin "C19")
+    (pin "C20")
+    (pin "D10")
+    (pin "D11")
+    (pin "D12")
+    (pin "D13")
+    (pin "D14")
+    (pin "D15")
+    (pin "D16")
+    (pin "D17")
+    (pin "D18")
+    (pin "D19")
+    (pin "D20")
+    (pin "E10")
+    (pin "E11")
+    (pin "E12")
+    (pin "E13")
+    (pin "E14")
+    (pin "E15")
+    (pin "E16")
+    (pin "E17")
+    (pin "E18")
+    (pin "E19")
+    (pin "E20")
+    (pin "F10")
+    (pin "F11")
+    (pin "F12")
+    (pin "F13")
+    (pin "F14")
+    (pin "F15")
+    (pin "F16")
+    (pin "F17")
+    (pin "F18")
+    (pin "F19")
+    (pin "F20")
+    (pin "G10")
+    (pin "G11")
+    (pin "G12")
+    (pin "G13")
+    (pin "G14")
+    (pin "G15")
+    (pin "G16")
+    (pin "G17")
+    (pin "G18")
+    (pin "G19")
+    (pin "G20")
+    (pin "H10")
+    (pin "H11")
+    (pin "H12")
+    (pin "H13")
+    (pin "H14")
+    (pin "H15")
+    (pin "H16")
+    (pin "H17")
+    (pin "H18")
+    (pin "H19")
+    (pin "H20")
+    (pin "J10")
+    (pin "J11")
+    (pin "J12")
+    (pin "J13")
+    (pin "J14")
+    (pin "J15")
+    (pin "J16")
+    (pin "J17")
+    (pin "J18")
+    (pin "J19")
+    (pin "J20")
+    (pin "K10")
+    (pin "K11")
+    (pin "K12")
+    (pin "K13")
+    (pin "K14")
+    (pin "K15")
+    (pin "K16")
+    (pin "K17")
+    (pin "K18")
+    (pin "K19")
+    (pin "K20")
+    (pin "L10")
+    (pin "L11")
+    (pin "L12")
+    (pin "L13")
+    (pin "L14")
+    (pin "L15")
+    (pin "L16")
+    (pin "L17")
+    (pin "L18")
+    (pin "L19")
+    (instances
+      (project "protoflow"
+        (path "/" (reference "U1") (unit 3))
+      )
+    )
+  )
   (sheet_instances
