File: hardware/prism_powerboard/PRISM_Power/untitled.kicad_sch (KiCad schematic)
At the start: 3 parts, among them U4 MAX17048G+T10

Commit message: Finished Schematics and Start Routing
Finished Schematics and started routing the PCB lines. Added and ensured all footprints were accurate
Parts:
- C7: footprint (none) -> Capacitor_SMD:C_0805_2012Metric_Pad1.18x1.45mm_HandSolder
- R1: value R -> 10k; footprint (none) -> Resistor_SMD:R_0805_2012Metric_Pad1.20x1.40mm_HandSolder
- U4: footprint 21-0168E_T822-3_MXM -> MAX17048G:21-0168E_T822-3_MXM
Changed lines of the file:
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@@
 			)
 		)
-		(property "Value" "R"
+		(property "Value" "10k"
 			(at 184.15 100.33 90)
 			(show_name no)
@@
 			)
 		)
-		(property "Footprint" ""
+		(property "Footprint" "Resistor_SMD:R_0805_2012Metric_Pad1.20x1.40mm_HandSolder"
 			(at 184.15 105.918 90)
 			(hide yes)
@@
 			)
 		)
-		(property "Footprint" ""
+		(property "Footprint" "Capacitor_SMD:C_0805_2012Metric_Pad1.18x1.45mm_HandSolder"
 			(at 110.1852 95.25 0)
 			(hide yes)
@@
 			)
 		)
-		(property "Footprint" "21-0168E_T822-3_MXM"
+		(property "Footprint" "MAX17048G:21-0168E_T822-3_MXM"
 			(at 118.11 82.55 0)
 			(hide yes)
