File: hardware/prism_powerboard/PRISM_Power/LP87563W_Q1.kicad_sch (KiCad schematic)
At the start: 20 parts, among them IC2 LP87564WRNFTQ1

Commit message: Finished Schematics and Start Routing
Finished Schematics and started routing the PCB lines. Added and ensured all footprints were accurate
Parts:
- IC2: footprint LP87524TRNFRQ1 -> LP87564RNFRQ1:RNF0026C
- R3: footprint (none) -> Resistor_SMD:R_0805_2012Metric_Pad1.20x1.40mm_HandSolder
Connections:
- net VANA renamed SYS_3V5
Changed lines of the file:
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@@
+		)
+	)
+	(global_label "SYS_3V5"
+		(shape input)
+		(at 54.61 90.17 180)
+		(fields_autoplaced yes)
+		(effects
+			(font
+				(size 1.27 1.27)
+			)
+			(justify right)
+		)
+		(property "Intersheetrefs" "${INTERSHEET_REFS}"
+			(at 43.642 90.17 0)
+			(hide yes)
+			(show_name no)
+			(do_not_autoplace no)
+			(effects
+				(font
+					(size 1.27 1.27)
+				)
+				(justify right)
+			)
 		)
 	)
@@
 		)
 	)
-	(global_label "VCC_Batt"
-		(shape input)
-		(at 54.61 74.93 180)
+	(global_label "FB_BO"
+		(shape input)
+		(at 182.88 40.64 90)
+		(fields_autoplaced yes)
+		(effects
+			(font
+				(size 1.27 1.27)
+			)
+			(justify left)
+		)
+		(property "Intersheetrefs" "${INTERSHEET_REFS}"
+			(at 182.88 31.7281 90)
+			(hide yes)
+			(show_name no)
+			(do_not_autoplace no)
+			(effects
+				(font
+					(size 1.27 1.27)
+				)
+				(justify left)
+			)
+		)
+	)
+	(global_label "Vin_B0"
+		(shape input)
+		(at 64.77 27.94 0)
+		(fields_autoplaced yes)
+		(effects
+			(font
+				(size 1.27 1.27)
+			)
+			(justify left)
+		)
+		(property "Intersheetrefs" "${INTERSHEET_REFS}"
+			(at 74.0447 27.94 0)
+			(hide yes)
+			(show_name no)
+			(do_not_autoplace no)
+			(effects
+				(font
+					(size 1.27 1.27)
+				)
+				(justify left)
+			)
+		)
+	)
+	(global_label "Vin_B0"
+		(shape input)
+		(at 100.33 38.1 180)
 		(fields_autoplaced yes)
 		(effects
@@
 		)
 		(property "Intersheetrefs" "${INTERSHEET_REFS}"
-			(at 43.1582 74.93 0)
-			(hide yes)
-			(show_name no)
-			(do_not_autoplace no)
-			(effects
-				(font
-					(size 1.27 1.27)
-				)
-				(justify right)
-			)
-		)
-	)
-	(global_label "FB_BO"
-		(shape input)
-		(at 182.88 40.64 90)
-		(fields_autoplaced yes)
-		(effects
-			(font
-				(size 1.27 1.27)
-			)
-			(justify left)
-		)
-		(property "Intersheetrefs" "${INTERSHEET_REFS}"
-			(at 182.88 31.7281 90)
-			(hide yes)
-			(show_name no)
-			(do_not_autoplace no)
-			(effects
-				(font
-					(size 1.27 1.27)
-				)
-				(justify left)
-			)
-		)
-	)
-	(global_label "Vin_B0"
-		(shape input)
-		(at 64.77 27.94 0)
-		(fields_autoplaced yes)
-		(effects
-			(font
-				(size 1.27 1.27)
-			)
-			(justify left)
-		)
-		(property "Intersheetrefs" "${INTERSHEET_REFS}"
-			(at 74.0447 27.94 0)
-			(hide yes)
-			(show_name no)
-			(do_not_autoplace no)
-			(effects
-				(font
-					(size 1.27 1.27)
-				)
-				(justify left)
-			)
-		)
-	)
-	(global_label "Vin_B0"
-		(shape input)
-		(at 100.33 38.1 180)
+			(at 91.0553 38.1 0)
+			(hide yes)
+			(show_name no)
+			(do_not_autoplace no)
+			(effects
+				(font
+					(size 1.27 1.27)
+				)
+				(justify right)
+			)
+		)
+	)
+	(global_label "CLK_IN_PS"
+		(shape input)
+		(at 100.33 60.96 180)
 		(fields_autoplaced yes)
 		(effects
@@
 		)
 		(property "Intersheetrefs" "${INTERSHEET_REFS}"
-			(at 91.0553 38.1 0)
-			(hide yes)
-			(show_name no)
-			(do_not_autoplace no)
-			(effects
-				(font
-					(size 1.27 1.27)
-				)
-				(justify right)
-			)
-		)
-	)
-	(global_label "CLK_IN_PS"
-		(shape input)
-		(at 100.33 60.96 180)
+			(at 87.4267 60.96 0)
+			(hide yes)
+			(show_name no)
+			(do_not_autoplace no)
+			(effects
+				(font
+					(size 1.27 1.27)
+				)
+				(justify right)
+			)
+		)
+	)
+	(global_label "SYS_3V5"
+		(shape input)
+		(at 54.61 27.94 180)
 		(fields_autoplaced yes)
 		(effects
@@
 		)
 		(property "Intersheetrefs" "${INTERSHEET_REFS}"
-			(at 87.4267 60.96 0)
+			(at 43.642 27.94 0)
 			(hide yes)
 			(show_name no)
@@
 		)
 	)
+	(global_label "SYS_3V5"
+		(shape input)
+		(at 54.61 74.93 180)
+		(fields_autoplaced yes)
+		(effects
+			(font
+				(size 1.27 1.27)
+			)
+			(justify right)
+		)
+		(property "Intersheetrefs" "${INTERSHEET_REFS}"
+			(at 43.642 74.93 0)
+			(hide yes)
+			(show_name no)
+			(do_not_autoplace no)
+			(effects
+				(font
+					(size 1.27 1.27)
+				)
+				(justify right)
+			)
+		)
+	)
 	(global_label "SDA"
 		(shape input)
@@
 		)
 	)
+	(global_label "SYS_3V5"
+		(shape input)
+		(at 54.61 59.69 180)
+		(fields_autoplaced yes)
+		(effects
+			(font
+				(size 1.27 1.27)
+			)
+			(justify right)
+		)
+		(property "Intersheetrefs" "${INTERSHEET_REFS}"
+			(at 43.642 59.69 0)
+			(hide yes)
+			(show_name no)
+			(do_not_autoplace no)
+			(effects
+				(font
+					(size 1.27 1.27)
+				)
+				(justify right)
+			)
+		)
+	)
 	(global_label "SW_B2"
 		(shape input)
@@
 		)
 	)
-	(global_label "VCC_Batt"
-		(shape input)
-		(at 54.61 44.45 180)
-		(fields_autoplaced yes)
-		(effects
-			(font
-				(size 1.27 1.27)
-			)
-			(justify right)
-		)
-		(property "Intersheetrefs" "${INTERSHEET_REFS}"
-			(at 43.1582 44.45 0)
-			(hide yes)
-			(show_name no)
-			(do_not_autoplace no)
-			(effects
-				(font
-					(size 1.27 1.27)
-				)
-				(justify right)
-			)
-		)
-	)
 	(global_label "FB_B1"
 		(shape input)
@@
 		)
 	)
-	(global_label "VCC_Batt"
-		(shape input)
-		(at 54.61 27.94 180)
-		(fields_autoplaced yes)
-		(effects
-			(font
-				(size 1.27 1.27)
-			)
-			(justify right)
-		)
-		(property "Intersheetrefs" "${INTERSHEET_REFS}"
-			(at 43.1582 27.94 0)
-			(hide yes)
-			(show_name no)
-			(do_not_autoplace no)
-			(effects
-				(font
-					(size 1.27 1.27)
-				)
-				(justify right)
-			)
-		)
-	)
 	(global_label "PGD_S"
 		(shape input)
@@
 		)
 	)
-	(global_label "VCC_Batt"
-		(shape input)
-		(at 54.61 59.69 180)
+	(global_label "SCL"
+		(shape input)
+		(at 100.33 58.42 180)
 		(fields_autoplaced yes)
 		(effects
@@
 		)
 		(property "Intersheetrefs" "${INTERSHEET_REFS}"
-			(at 43.1582 59.69 0)
-			(hide yes)
-			(show_name no)
-			(do_not_autoplace no)
-			(effects
-				(font
-					(size 1.27 1.27)
-				)
-				(justify right)
-			)
-		)
-	)
-	(global_label "SCL"
-		(shape input)
-		(at 100.33 58.42 180)
-		(fields_autoplaced yes)
-		(effects
-			(font
-				(size 1.27 1.27)
-			)
-			(justify right)
-		)
-		(property "Intersheetrefs" "${INTERSHEET_REFS}"
 			(at 93.8372 58.42 0)
-			(hide yes)
-			(show_name no)
-			(do_not_autoplace no)
-			(effects
-				(font
-					(size 1.27 1.27)
-				)
-				(justify right)
-			)
-		)
-	)
-	(global_label "VCC_Batt"
-		(shape input)
-		(at 54.61 90.17 180)
-		(fields_autoplaced yes)
-		(effects
-			(font
-				(size 1.27 1.27)
-			)
-			(justify right)
-		)
-		(property "Intersheetrefs" "${INTERSHEET_REFS}"
-			(at 43.1582 90.17 0)
 			(hide yes)
 			(show_name no)
@@
 		(property "Intersheetrefs" "${INTERSHEET_REFS}"
 			(at 91.0553 40.64 0)
+			(hide yes)
+			(show_name no)
+			(do_not_autoplace no)
+			(effects
+				(font
+					(size 1.27 1.27)
+				)
+				(justify right)
+			)
+		)
+	)
+	(global_label "SYS_3V5"
+		(shape input)
+		(at 54.61 44.45 180)
+		(fields_autoplaced yes)
+		(effects
+			(font
+				(size 1.27 1.27)
+			)
+			(justify right)
+		)
+		(property "Intersheetrefs" "${INTERSHEET_REFS}"
+			(at 43.642 44.45 0)
 			(hide yes)
 			(show_name no)
@@
 			)
 		)
-		(property "Footprint" "LP87524TRNFRQ1"
+		(property "Footprint" "LP87564RNFRQ1:RNF0026C"
 			(at 134.62 133.02 0)
 			(hide yes)
@@
 			)
 		)
-		(property "Footprint" ""
+		(property "Footprint" "Resistor_SMD:R_0805_2012Metric_Pad1.20x1.40mm_HandSolder"
 			(at 80.772 68.58 90)
 			(hide yes)

Commit message: PCB Routing
More PCB Routing and organizing components. Also fixed PMIC wrong Voltage labels/nets.
Connections:
- removed net +1V8: C18.1, C19.1, C20.1, C43.1, C44.1, C45.1, C46.1, C47.1, IC2.1 (FB_B2_1), IC2.14 (FB_B1_1), IC2.21 (FB_B3_1), IC2.8 (FB_B0_1), L5.2, L6.2, L7.2, L8.2
- net SCL renamed I2C_SCL_1V8
- net SDA renamed I2C_SDA_1V8
- new net +1V0: C18.1, C20.1, IC2.8 (FB_B0_1), L5.2
- new net +1V35: C44.1, C45.1, IC2.1 (FB_B2_1), L7.2
- new net +1V8_PMIC: C19.1, C43.1, IC2.14 (FB_B1_1), L6.2
- new net +2V1: C46.1, C47.1, IC2.21 (FB_B3_1), L8.2
